Commit message: feat(urdf): un origin por junta con meshes sin origin y pinza fija
Los visuales pasan a meshes STL ya colocados en el marco de cada eslabon,
eliminando los origin dentro de <visual>. Se acopla la pinza a tool0 con
gripper_mount y gripper_tcp_joint (juntas fijas, sin grados de libertad).

Co-Authored-By: Claude Sonnet 5.5 <noreply@anthropic.com>

File: 2-2026/IMT342/equipo/proyecto/ros2_ws/src/irb120_hito1/urdf/irb120.macro.xacro (robot description, xacro)
@@ -2,6 +2,8 @@
 <robot xmlns:xacro="http://www.ros.org/wiki/xacro">
   <!--
-    Cadena cinemática mínima: seis juntas revolutas y seis marcos móviles.
-    base_link es el marco base y no cuenta como una de las seis juntas.
+    Seis juntas revolutas (un único origin por grado de libertad) y seis marcos
+    móviles. base_link es el marco base y no cuenta como junta. Los visuales son
+    meshes STL ya expresados en el marco de su eslabón: no llevan origin propio.
+    La pinza se acopla a tool0 con dos juntas fijas (no son grados de libertad).
     Para DH clásico A_i(q_i)=Rz(q_i) B_i, donde
     B_i=Tz(d_i) Tx(a_i) Rx(alpha_i). URDF aplica en cada junta
@@ -11,9 +13,9 @@
     Tz(d6) conmuta con Rz(q6). Así, tool0 es directamente el hijo de joint_6.
   -->
+  <xacro:property name="gripper_tcp_z" value="0.100"/>
   <xacro:macro name="irb120_robot" params="prefix:=''">
     <link name="${prefix}base_link">
       <visual>
-        <origin xyz="0 0 0.0935" rpy="0 0 0"/>
-        <geometry><cylinder radius="0.09" length="0.187"/></geometry>
+        <geometry><mesh filename="package://irb120_hito1/meshes/base_link.stl"/></geometry>
         <material name="abb_dark"/>
       </visual>
@@ -22,6 +24,5 @@
     <link name="${prefix}link_1">
       <visual>
-        <origin xyz="0 0 0.145" rpy="0 0 0"/>
-        <geometry><cylinder radius="0.055" length="0.290"/></geometry>
+        <geometry><mesh filename="package://irb120_hito1/meshes/link_1.stl"/></geometry>
         <material name="abb_orange"/>
       </visual>
@@ -37,6 +38,5 @@
     <link name="${prefix}link_2">
       <visual>
-        <origin xyz="0.135 0 0" rpy="0 0 0"/>
-        <geometry><box size="0.270 0.075 0.075"/></geometry>
+        <geometry><mesh filename="package://irb120_hito1/meshes/link_2.stl"/></geometry>
         <material name="abb_orange"/>
       </visual>
@@ -52,6 +52,5 @@
     <link name="${prefix}link_3">
       <visual>
-        <origin xyz="0.035 0 0" rpy="0 0 0"/>
-        <geometry><box size="0.070 0.070 0.070"/></geometry>
+        <geometry><mesh filename="package://irb120_hito1/meshes/link_3.stl"/></geometry>
         <material name="abb_orange"/>
       </visual>
@@ -67,6 +66,5 @@
     <link name="${prefix}link_4">
       <visual>
-        <origin xyz="0 0 0.151" rpy="0 0 0"/>
-        <geometry><cylinder radius="0.045" length="0.302"/></geometry>
+        <geometry><mesh filename="package://irb120_hito1/meshes/link_4.stl"/></geometry>
         <material name="abb_orange"/>
       </visual>
@@ -82,6 +80,5 @@
     <link name="${prefix}link_5">
       <visual>
-        <origin xyz="0 0.036 0" rpy="${-pi/2} 0 0"/>
-        <geometry><cylinder radius="0.035" length="0.072"/></geometry>
+        <geometry><mesh filename="package://irb120_hito1/meshes/link_5.stl"/></geometry>
         <material name="abb_orange"/>
       </visual>
@@ -97,6 +94,5 @@
     <link name="${prefix}tool0">
       <visual>
-        <origin xyz="0 0 -0.009" rpy="0 0 0"/>
-        <geometry><cylinder radius="0.032" length="0.018"/></geometry>
+        <geometry><mesh filename="package://irb120_hito1/meshes/tool0.stl"/></geometry>
         <material name="metal"/>
       </visual>
@@ -109,4 +105,22 @@
       <limit lower="-6.9813170080" upper="6.9813170080" effort="100" velocity="7.3303828584"/>
     </joint>
+    <!-- Pinza neumática: gripper_link comparte el marco de tool0 (sin origin). -->
+    <link name="${prefix}gripper_link">
+      <visual>
+        <geometry><mesh filename="package://irb120_hito1/meshes/gripper_link.stl"/></geometry>
+        <material name="abb_dark"/>
+      </visual>
+    </link>
+    <joint name="${prefix}gripper_mount" type="fixed">
+      <parent link="${prefix}tool0"/>
+      <child link="${prefix}gripper_link"/>
+    </joint>
+    <!-- TCP: centro de agarre entre los dedos, 0.100 m sobre la brida. -->
+    <link name="${prefix}gripper_tcp"/>
+    <joint name="${prefix}gripper_tcp_joint" type="fixed">
+      <parent link="${prefix}gripper_link"/>
+      <child link="${prefix}gripper_tcp"/>
+      <origin xyz="0 0 ${gripper_tcp_z}"/>
+    </joint>
   </xacro:macro>
 </robot>

File: 2-2026/IMT342/equipo/proyecto/ros2_ws/src/irb120_hito1/urdf/irb120.urdf (robot description, URDF)
Before this commit: robot irb120_hito1, 7 links, 6 joints
Links:
- added link gripper_link; visual mesh filename=package://irb120_hito1/meshes/gripper_link.stl
- added link gripper_tcp
- link base_link: geometry visual mesh filename=package://irb120_hito1/meshes/base_link.stl
- link link_1: geometry visual mesh filename=package://irb120_hito1/meshes/link_1.stl
- link link_2: geometry visual mesh filename=package://irb120_hito1/meshes/link_2.stl
- link link_3: geometry visual mesh filename=package://irb120_hito1/meshes/link_3.stl
- link link_4: geometry visual mesh filename=package://irb120_hito1/meshes/link_4.stl
- link link_5: geometry visual mesh filename=package://irb120_hito1/meshes/link_5.stl
- link tool0: geometry visual mesh filename=package://irb120_hito1/meshes/tool0.stl
Joints:
- added joint gripper_mount: type fixed, parent tool0, child gripper_link
- added joint gripper_tcp_joint: type fixed, parent gripper_link, child gripper_tcp, origin xyz=0 0 0.1

Commit message: feat(cad): CAD real del IRB 120 como visual y collision, con verificador de colisiones
Importa los STL de ROS-Industrial (Apache-2.0) a los marcos del URDF con
scripts/import_cad.py y agrega bloques collision. irb120_hito2 incorpora
CollisionChecker (autocolision y mesa) y el nodo IK descarta soluciones en
colision. Actualiza pruebas y documentacion; 38 pruebas aprobadas.

Co-Authored-By: Claude Sonnet 5.5 <noreply@anthropic.com>

File: 2-2026/IMT342/equipo/proyecto/ros2_ws/src/irb120_hito1/urdf/irb120.macro.xacro (robot description, xacro)
@@ -3,6 +3,7 @@
   <!--
     Seis juntas revolutas (un único origin por grado de libertad) y seis marcos
-    móviles. base_link es el marco base y no cuenta como junta. Los visuales son
-    meshes STL ya expresados en el marco de su eslabón: no llevan origin propio.
+    móviles. base_link es el marco base y no cuenta como junta. Visual y collision
+    son meshes STL del CAD real (ROS-Industrial, Apache-2.0) ya expresados en el
+    marco de su eslabón: no llevan origin propio.
     La pinza se acopla a tool0 con dos juntas fijas (no son grados de libertad).
     Para DH clásico A_i(q_i)=Rz(q_i) B_i, donde
@@ -17,14 +18,20 @@
     <link name="${prefix}base_link">
       <visual>
-        <geometry><mesh filename="package://irb120_hito1/meshes/base_link.stl"/></geometry>
+        <geometry><mesh filename="package://irb120_hito1/meshes/visual/base_link.stl"/></geometry>
         <material name="abb_dark"/>
       </visual>
+      <collision>
+        <geometry><mesh filename="package://irb120_hito1/meshes/collision/base_link.stl"/></geometry>
+      </collision>
     </link>
     <!-- J1: O1=I. -->
     <link name="${prefix}link_1">
       <visual>
-        <geometry><mesh filename="package://irb120_hito1/meshes/link_1.stl"/></geometry>
+        <geometry><mesh filename="package://irb120_hito1/meshes/visual/link_1.stl"/></geometry>
         <material name="abb_orange"/>
       </visual>
+      <collision>
+        <geometry><mesh filename="package://irb120_hito1/meshes/collision/link_1.stl"/></geometry>
+      </collision>
     </link>
     <joint name="${prefix}joint_1" type="revolute">
@@ -38,7 +45,10 @@
     <link name="${prefix}link_2">
       <visual>
-        <geometry><mesh filename="package://irb120_hito1/meshes/link_2.stl"/></geometry>
+        <geometry><mesh filename="package://irb120_hito1/meshes/visual/link_2.stl"/></geometry>
         <material name="abb_orange"/>
       </visual>
+      <collision>
+        <geometry><mesh filename="package://irb120_hito1/meshes/collision/link_2.stl"/></geometry>
+      </collision>
     </link>
     <joint name="${prefix}joint_2" type="revolute">
@@ -52,7 +62,10 @@
     <link name="${prefix}link_3">
       <visual>
-        <geometry><mesh filename="package://irb120_hito1/meshes/link_3.stl"/></geometry>
+        <geometry><mesh filename="package://irb120_hito1/meshes/visual/link_3.stl"/></geometry>
         <material name="abb_orange"/>
       </visual>
+      <collision>
+        <geometry><mesh filename="package://irb120_hito1/meshes/collision/link_3.stl"/></geometry>
+      </collision>
     </link>
     <joint name="${prefix}joint_3" type="revolute">
@@ -66,7 +79,10 @@
     <link name="${prefix}link_4">
       <visual>
-        <geometry><mesh filename="package://irb120_hito1/meshes/link_4.stl"/></geometry>
+        <geometry><mesh filename="package://irb120_hito1/meshes/visual/link_4.stl"/></geometry>
         <material name="abb_orange"/>
       </visual>
+      <collision>
+        <geometry><mesh filename="package://irb120_hito1/meshes/collision/link_4.stl"/></geometry>
+      </collision>
     </link>
     <joint name="${prefix}joint_4" type="revolute">
@@ -80,7 +96,10 @@
     <link name="${prefix}link_5">
       <visual>
-        <geometry><mesh filename="package://irb120_hito1/meshes/link_5.stl"/></geometry>
+        <geometry><mesh filename="package://irb120_hito1/meshes/visual/link_5.stl"/></geometry>
         <material name="abb_orange"/>
       </visual>
+      <collision>
+        <geometry><mesh filename="package://irb120_hito1/meshes/collision/link_5.stl"/></geometry>
+      </collision>
     </link>
     <joint name="${prefix}joint_5" type="revolute">
@@ -94,7 +113,10 @@
     <link name="${prefix}tool0">
       <visual>
-        <geometry><mesh filename="package://irb120_hito1/meshes/tool0.stl"/></geometry>
+        <geometry><mesh filename="package://irb120_hito1/meshes/visual/tool0.stl"/></geometry>
         <material name="metal"/>
       </visual>
+      <collision>
+        <geometry><mesh filename="package://irb120_hito1/meshes/collision/tool0.stl"/></geometry>
+      </collision>
     </link>
     <joint name="${prefix}joint_6" type="revolute">
@@ -108,7 +130,10 @@
     <link name="${prefix}gripper_link">
       <visual>
-        <geometry><mesh filename="package://irb120_hito1/meshes/gripper_link.stl"/></geometry>
+        <geometry><mesh filename="package://irb120_hito1/meshes/visual/gripper_link.stl"/></geometry>
         <material name="abb_dark"/>
       </visual>
+      <collision>
+        <geometry><mesh filename="package://irb120_hito1/meshes/collision/gripper_link.stl"/></geometry>
+      </collision>
     </link>
     <joint name="${prefix}gripper_mount" type="fixed">

File: 2-2026/IMT342/equipo/proyecto/ros2_ws/src/irb120_hito1/urdf/irb120.urdf (robot description, URDF)
Before this commit: robot irb120_hito1, 9 links, 8 joints
Links:
- link base_link: geometry collision mesh filename=package://irb120_hito1/meshes/collision/base_link.stl; visual mesh filename=package://irb120_hito1/meshes/visual/base_link.stl
- link gripper_link: geometry collision mesh filename=package://irb120_hito1/meshes/collision/gripper_link.stl; visual mesh filename=package://irb120_hito1/meshes/visual/gripper_link.stl
- link link_1: geometry collision mesh filename=package://irb120_hito1/meshes/collision/link_1.stl; visual mesh filename=package://irb120_hito1/meshes/visual/link_1.stl
- link link_2: geometry collision mesh filename=package://irb120_hito1/meshes/collision/link_2.stl; visual mesh filename=package://irb120_hito1/meshes/visual/link_2.stl
- link link_3: geometry collision mesh filename=package://irb120_hito1/meshes/collision/link_3.stl; visual mesh filename=package://irb120_hito1/meshes/visual/link_3.stl
- link link_4: geometry collision mesh filename=package://irb120_hito1/meshes/collision/link_4.stl; visual mesh filename=package://irb120_hito1/meshes/visual/link_4.stl
- link link_5: geometry collision mesh filename=package://irb120_hito1/meshes/collision/link_5.stl; visual mesh filename=package://irb120_hito1/meshes/visual/link_5.stl
- link tool0: geometry collision mesh filename=package://irb120_hito1/meshes/collision/tool0.stl; visual mesh filename=package://irb120_hito1/meshes/visual/tool0.stl
