Commit message: Actualizacion de hito 1 con las correcciones

File: 2-2026/IMT342/equipo/proyecto/ros2_ws/src/irb120_hito1/urdf/irb120.macro.xacro (robot description, xacro)
@@ -2,7 +2,12 @@
 <robot xmlns:xacro="http://www.ros.org/wiki/xacro">
   <!--
-    Cadena canonica del IRB 120 basada en DH clasico.
-    Cada fila se separa en: Rz(q_i), Rz(offset_i), Tz(d_i) Tx(a_i) Rx(alpha_i).
-    Esta separacion evita esconder offsets en los valores publicados por /joint_states.
+    Cadena cinemática mínima: seis juntas revolutas y seis marcos móviles.
+    base_link es el marco base y no cuenta como una de las seis juntas.
+    Para DH clásico A_i(q_i)=Rz(q_i) B_i, donde
+    B_i=Tz(d_i) Tx(a_i) Rx(alpha_i). URDF aplica en cada junta
+    O_i Rz(q_i), por lo que el B de una fila se incorpora al origin de la
+    junta siguiente. Los offsets de theta también se incluyen en esos origins.
+    La sexta fila puede cerrarse sin una junta fija porque a6=alpha6=0 y
+    Tz(d6) conmuta con Rz(q6). Así, tool0 es directamente el hijo de joint_6.
   -->
   <xacro:macro name="irb120_robot" params="prefix:=''">
@@ -13,11 +18,7 @@
         <material name="abb_dark"/>
       </visual>
-      <collision>
-        <origin xyz="0 0 0.0935" rpy="0 0 0"/>
-        <geometry><cylinder radius="0.09" length="0.187"/></geometry>
-      </collision>
     </link>
-    <!-- Fila DH 1: d=0.290, a=0, alpha=-pi/2. -->
-    <link name="${prefix}joint_1_frame">
+    <!-- J1: O1=I. -->
+    <link name="${prefix}link_1">
       <visual>
         <origin xyz="0 0 0.145" rpy="0 0 0"/>
@@ -28,38 +29,11 @@
     <joint name="${prefix}joint_1" type="revolute">
       <parent link="${prefix}base_link"/>
-      <child link="${prefix}joint_1_frame"/>
+      <child link="${prefix}link_1"/>
+      <origin xyz="0 0 0" rpy="0 0 0"/>
       <axis xyz="0 0 1"/>
       <limit lower="-2.8797932658" upper="2.8797932658" effort="100" velocity="4.3633231300"/>
     </joint>
-    <link name="${prefix}theta_1_frame"/>
-    <joint name="${prefix}theta_offset_1" type="fixed">
-      <parent link="${prefix}joint_1_frame"/>
-      <child link="${prefix}theta_1_frame"/>
-    </joint>
-    <link name="${prefix}link_1">
-      <inertial>
-        <origin xyz="0 0.054 0" rpy="0 0 0"/>
-        <mass value="4.248"/>
-        <inertia ixx="0.019699" ixy="0" ixz="0" iyy="0.014484" iyz="0" izz="0.019952"/>
-      </inertial>
-      <visual>
-        <geometry><sphere radius="0.065"/></geometry>
-        <material name="abb_orange"/>
-      </visual>
-    </link>
-    <joint name="${prefix}dh_1" type="fixed">
-      <parent link="${prefix}theta_1_frame"/>
-      <child link="${prefix}link_1"/>
-      <origin xyz="0 0 0.290" rpy="${-pi/2} 0 0"/>
-    </joint>
-    <!-- Fila DH 2: theta=q2-pi/2, d=0, a=0.270, alpha=0. -->
-    <link name="${prefix}joint_2_frame"/>
-    <joint name="${prefix}joint_2" type="revolute">
-      <parent link="${prefix}link_1"/>
-      <child link="${prefix}joint_2_frame"/>
-      <axis xyz="0 0 1"/>
-      <limit lower="-1.9198621772" upper="1.9198621772" effort="100" velocity="4.3633231300"/>
-    </joint>
-    <link name="${prefix}theta_2_frame">
+    <!-- J2: O2=B1 Rz(-pi/2). -->
+    <link name="${prefix}link_2">
       <visual>
         <origin xyz="0.135 0 0" rpy="0 0 0"/>
@@ -68,31 +42,13 @@
       </visual>
     </link>
-    <joint name="${prefix}theta_offset_2" type="fixed">
-      <parent link="${prefix}joint_2_frame"/>
-      <child link="${prefix}theta_2_frame"/>
-      <origin xyz="0 0 0" rpy="0 0 ${-pi/2}"/>
+    <joint name="${prefix}joint_2" type="revolute">
+      <parent link="${prefix}link_1"/>
+      <child link="${prefix}link_2"/>
+      <origin xyz="0 0 0.290" rpy="${-pi/2} ${-pi/2} 0"/>
+      <axis xyz="0 0 1"/>
+      <limit lower="-1.9198621772" upper="1.9198621772" effort="100" velocity="4.3633231300"/>
     </joint>
-    <link name="${prefix}link_2">
-      <inertial>
-        <origin xyz="-0.169 0 0" rpy="0 0 0"/>
-        <mass value="5.412"/>
-        <inertia ixx="0.035942" ixy="0" ixz="0" iyy="0.083522" iyz="0" izz="0.057569"/>
-      </inertial>
-      <visual><geometry><sphere radius="0.060"/></geometry><material name="abb_orange"/></visual>
-    </link>
-    <joint name="${prefix}dh_2" type="fixed">
-      <parent link="${prefix}theta_2_frame"/>
-      <child link="${prefix}link_2"/>
-      <origin xyz="0.270 0 0" rpy="0 0 0"/>
-    </joint>
-    <!-- Fila DH 3: d=0, a=0.070, alpha=-pi/2. -->
-    <link name="${prefix}joint_3_frame"/>
-    <joint name="${prefix}joint_3" type="revolute">
-      <parent link="${prefix}link_2"/>
-      <child link="${prefix}joint_3_frame"/>
-      <axis xyz="0 0 1"/>
-      <limit lower="-1.9198621772" upper="1.2217304764" effort="100" velocity="4.3633231300"/>
-    </joint>
-    <link name="${prefix}theta_3_frame">
+    <!-- J3: O3=B2=Tx(0.270). -->
+    <link name="${prefix}link_3">
       <visual>
         <origin xyz="0.035 0 0" rpy="0 0 0"/>
@@ -101,30 +57,13 @@
       </visual>
     </link>
-    <joint name="${prefix}theta_offset_3" type="fixed">
-      <parent link="${prefix}joint_3_frame"/>
-      <child link="${prefix}theta_3_frame"/>
+    <joint name="${prefix}joint_3" type="revolute">
+      <parent link="${prefix}link_2"/>
+      <child link="${prefix}link_3"/>
+      <origin xyz="0.270 0 0" rpy="0 0 0"/>
+      <axis xyz="0 0 1"/>
+      <limit lower="-1.9198621772" upper="1.2217304764" effort="100" velocity="4.3633231300"/>
     </joint>
-    <link name="${prefix}link_3">
-      <inertial>
-        <origin xyz="-0.012 0 0.023" rpy="0 0 0"/>
-        <mass value="4.077"/>
-        <inertia ixx="0.017562" ixy="0" ixz="-0.001993" iyy="0.023140" iyz="0" izz="0.011589"/>
-      </inertial>
-      <visual><geometry><sphere radius="0.055"/></geometry><material name="abb_orange"/></visual>
-    </link>
-    <joint name="${prefix}dh_3" type="fixed">
-      <parent link="${prefix}theta_3_frame"/>
-      <child link="${prefix}link_3"/>
-      <origin xyz="0.070 0 0" rpy="${-pi/2} 0 0"/>
-    </joint>
-    <!-- Fila DH 4: d=0.302, a=0, alpha=pi/2. -->
-    <link name="${prefix}joint_4_frame"/>
-    <joint name="${prefix}joint_4" type="revolute">
-      <parent link="${prefix}link_3"/>
-      <child link="${prefix}joint_4_frame"/>
-      <axis xyz="0 0 1"/>
-      <limit lower="-2.7925268032" upper="2.7925268032" effort="100" velocity="5.5850536064"/>
-    </joint>
-    <link name="${prefix}theta_4_frame">
+    <!-- J4: O4=B3=Tx(0.070) Rx(-pi/2). -->
+    <link name="${prefix}link_4">
       <visual>
         <origin xyz="0 0 0.151" rpy="0 0 0"/>
@@ -133,85 +72,41 @@
       </visual>
     </link>
-    <joint name="${prefix}theta_offset_4" type="fixed">
-      <parent link="${prefix}joint_4_frame"/>
-      <child link="${prefix}theta_4_frame"/>
+    <joint name="${prefix}joint_4" type="revolute">
+      <parent link="${prefix}link_3"/>
+      <child link="${prefix}link_4"/>
+      <origin xyz="0.070 0 0" rpy="${-pi/2} 0 0"/>
+      <axis xyz="0 0 1"/>
+      <limit lower="-2.7925268032" upper="2.7925268032" effort="100" velocity="5.5850536064"/>
     </joint>
-    <link name="${prefix}link_4">
-      <inertial>
-        <origin xyz="0 -0.007 0" rpy="0 0 0"/>
-        <mass value="1.832"/>
-        <inertia ixx="0.007247" ixy="0" ixz="0" iyy="0.003919" iyz="0" izz="0.005551"/>
-      </inertial>
-      <visual><geometry><sphere radius="0.045"/></geometry><material name="abb_orange"/></visual>
+    <!-- J5: O5=B4=Tz(0.302) Rx(pi/2). -->
+    <link name="${prefix}link_5">
+      <visual>
+        <origin xyz="0 0.036 0" rpy="${-pi/2} 0 0"/>
+        <geometry><cylinder radius="0.035" length="0.072"/></geometry>
+        <material name="abb_orange"/>
+      </visual>
     </link>
-    <joint name="${prefix}dh_4" type="fixed">
-      <parent link="${prefix}theta_4_frame"/>
-      <child link="${prefix}link_4"/>
-      <origin xyz="0 0 0.302" rpy="${pi/2} 0 0"/>
-    </joint>
-    <!-- Fila DH 5: d=0, a=0, alpha=-pi/2. -->
-    <link name="${prefix}joint_5_frame"/>
     <joint name="${prefix}joint_5" type="revolute">
       <parent link="${prefix}link_4"/>
-      <child link="${prefix}joint_5_frame"/>
+      <child link="${prefix}link_5"/>
+      <origin xyz="0 0 0.302" rpy="${pi/2} 0 0"/>
       <axis xyz="0 0 1"/>
       <limit lower="-2.0943951024" upper="2.0943951024" effort="100" velocity="5.5850536064"/>
     </joint>
-    <link name="${prefix}theta_5_frame"/>
-    <joint name="${prefix}theta_offset_5" type="fixed">
-      <parent link="${prefix}joint_5_frame"/>
-      <child link="${prefix}theta_5_frame"/>
-    </joint>
-    <link name="${prefix}link_5">
-      <inertial>
-        <origin xyz="0 0 0" rpy="0 0 0"/>
-        <mass value="0.755"/>
-        <inertia ixx="0.001120" ixy="0" ixz="0" iyy="0.001227" iyz="0" izz="0.000559"/>
-      </inertial>
-      <visual><geometry><sphere radius="0.035"/></geometry><material name="abb_orange"/></visual>
+    <!-- J6: O6=B5 Rz(pi) Tz(0.072). tool0 es el sexto marco móvil. -->
+    <link name="${prefix}tool0">
+      <visual>
+        <origin xyz="0 0 -0.009" rpy="0 0 0"/>
+        <geometry><cylinder radius="0.032" length="0.018"/></geometry>
+        <material name="metal"/>
+      </visual>
     </link>
-    <joint name="${prefix}dh_5" type="fixed">
-      <parent link="${prefix}theta_5_frame"/>
-      <child link="${prefix}link_5"/>
-      <origin xyz="0 0 0" rpy="${-pi/2} 0 0"/>
-    </joint>
-    <!-- Fila DH 6: theta=q6+pi, d=0.072, a=0, alpha=0. -->
-    <link name="${prefix}joint_6_frame"/>
     <joint name="${prefix}joint_6" type="revolute">
       <parent link="${prefix}link_5"/>
-      <child link="${prefix}joint_6_frame"/>
+      <child link="${prefix}tool0"/>
+      <origin xyz="0 0.072 0" rpy="${pi/2} 0 ${pi}"/>
       <axis xyz="0 0 1"/>
       <limit lower="-6.9813170080" upper="6.9813170080" effort="100" velocity="7.3303828584"/>
     </joint>
-    <link name="${prefix}theta_6_frame">
-      <visual>
-        <origin xyz="0 0 0.036" rpy="0 0 0"/>
-        <geometry><cylinder radius="0.028" length="0.072"/></geometry>
-        <material name="metal"/>
-      </visual>
-    </link>
-    <joint name="${prefix}theta_offset_6" type="fixed">
-      <parent link="${prefix}joint_6_frame"/>
-      <child link="${prefix}theta_6_frame"/>
-      <origin xyz="0 0 0" rpy="0 0 ${pi}"/>
-    </joint>
-    <link name="${prefix}link_6">
-      <inertial>
-        <origin xyz="0 0 -0.007" rpy="0 0 0"/>
-        <mass value="0.019"/>
-        <inertia ixx="0.000002347" ixy="0" ixz="0" iyy="0.000002347" iyz="0" izz="0.000004123"/>
-      </inertial>
-      <visual><geometry><cylinder radius="0.032" length="0.018"/></geometry><material name="metal"/></visual>
-    </link>
-    <joint name="${prefix}dh_6" type="fixed">
-      <parent link="${prefix}theta_6_frame"/>
-      <child link="${prefix}link_6"/>
-      <origin xyz="0 0 0.072" rpy="0 0 0"/>
-    </joint>
-    <link name="${prefix}tool0"/>
-    <joint name="${prefix}tool0_fixed" type="fixed">
-      <parent link="${prefix}link_6"/>
-      <child link="${prefix}tool0"/>
-    </joint>
   </xacro:macro>
 </robot>

File: 2-2026/IMT342/equipo/proyecto/ros2_ws/src/irb120_hito1/urdf/irb120.urdf.xacro (robot description, xacro)
@@ -3,7 +3,5 @@
   <xacro:include filename="$(find irb120_hito1)/urdf/materials.xacro"/>
   <xacro:include filename="$(find irb120_hito1)/urdf/irb120.macro.xacro"/>
-  <xacro:include filename="$(find irb120_hito1)/urdf/gripper.macro.xacro"/>
   <xacro:irb120_materials/>
   <xacro:irb120_robot/>
-  <xacro:parallel_gripper parent="tool0"/>
 </robot>

Commit message: feat(hito1): panel Qt con pasaporte en vivo, TCP unificado y bateria de pruebas
- Panel de control en Qt (el panel Tk no abria: tkinter no existe para el
  Python 3.12 de Jazzy). Deslizadores J1-J6, posturas, demo, pasaporte
  RViz (TF) vs DH con indicador frente a 1e-6 m y pestana de pruebas.
- TCP unico en config/tcp.yaml (0.150 m, no medido en el robot).
- Modulo validation.py compartido por verify_model y el panel (206 casos).
- Comparacion FK contra ROS-Industrial con evidencia CSV.
- 38 pruebas en irb120_hito1; se retira tests_require (aviso de colcon).
- Documentacion del Hito 1 auditada y actualizada.

File: 2-2026/IMT342/equipo/proyecto/ros2_ws/src/irb120_hito1/urdf/irb120.macro.xacro (robot description, xacro)
@@ -13,7 +13,8 @@
     La sexta fila puede cerrarse sin una junta fija porque a6=alpha6=0 y
     Tz(d6) conmuta con Rz(q6). Así, tool0 es directamente el hijo de joint_6.
+    gripper_tcp_z no tiene valor por defecto aquí: lo entrega irb120.urdf.xacro
+    desde config/tcp.yaml, la misma fuente que lee kinematics/dh.py.
   -->
-  <xacro:property name="gripper_tcp_z" value="0.100"/>
-  <xacro:macro name="irb120_robot" params="prefix:=''">
+  <xacro:macro name="irb120_robot" params="gripper_tcp_z prefix:=''">
     <link name="${prefix}base_link">
       <visual>
@@ -141,5 +142,6 @@
       <child link="${prefix}gripper_link"/>
     </joint>
-    <!-- TCP: centro de agarre entre los dedos, 0.100 m sobre la brida. -->
+    <!-- TCP: punto sobre el eje Z de tool0, gripper_tcp_z sobre la brida
+         (config/tcp.yaml; valor de modelo, no verificado en el robot). -->
     <link name="${prefix}gripper_tcp"/>
     <joint name="${prefix}gripper_tcp_joint" type="fixed">

File: 2-2026/IMT342/equipo/proyecto/ros2_ws/src/irb120_hito1/urdf/irb120.urdf (robot description, URDF)
Before this commit: robot irb120_hito1, 9 links, 8 joints
Joints:
- joint gripper_tcp_joint: origin xyz=0 0 0.1 -> xyz=0 0 0.15

File: 2-2026/IMT342/equipo/proyecto/ros2_ws/src/irb120_hito1/urdf/irb120.urdf.xacro (robot description, xacro)
@@ -1,7 +1,14 @@
 <?xml version="1.0"?>
 <robot name="irb120_hito1" xmlns:xacro="http://www.ros.org/wiki/xacro">
+  <!--
+    tcp_config: YAML con tool0_to_tcp_z_m. Es la fuente única del TCP; el mismo
+    archivo lo lee kinematics/dh.py. Para otra herramienta:
+      xacro irb120.urdf.xacro tcp_config:=/ruta/otra_pinza.yaml
+  -->
+  <xacro:arg name="tcp_config" default="$(find irb120_hito1)/config/tcp.yaml"/>
+  <xacro:property name="tcp" value="${xacro.load_yaml('$(arg tcp_config)')}"/>
   <xacro:include filename="$(find irb120_hito1)/urdf/materials.xacro"/>
   <xacro:include filename="$(find irb120_hito1)/urdf/irb120.macro.xacro"/>
   <xacro:irb120_materials/>
-  <xacro:irb120_robot/>
+  <xacro:irb120_robot gripper_tcp_z="${tcp['tool0_to_tcp_z_m']}"/>
 </robot>
